File: HW6/ME433-EAGLE/me433-2021-1.brd (EAGLE design)
At the start: 100 x 100 mm, 56 parts, among them J1 B, J2 A, U2 PIC32MX170F256B

Commit message: HW10
Parts:
- added B8, B9: (no value), ME433:1X01
Connections:
- net B15: now also B8.1, B9.1
Routing:
- net B15: track 87.7 -> 116.9 mm
Changed lines of the file:
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@@
 <attribute name="VALUE" x="45.212" y="2.54" size="0.6096" layer="27" font="vector" ratio="20" rot="R90"/>
+</element>
+<element name="B8" library="ME433" package="1X01" value="" x="5.08" y="7.62" smashed="yes">
+<attribute name="NAME" x="3.81" y="9.017" size="0.6096" layer="25" font="vector" ratio="20"/>
+<attribute name="VALUE" x="3.81" y="6.096" size="0.6096" layer="27" font="vector" ratio="20" align="top-left"/>
+</element>
+<element name="B9" library="ME433" package="1X01" value="" x="60.96" y="54.61" smashed="yes">
+<attribute name="NAME" x="59.69" y="56.007" size="0.6096" layer="25" font="vector" ratio="20"/>
+<attribute name="VALUE" x="59.69" y="53.086" size="0.6096" layer="27" font="vector" ratio="20" align="top-left"/>
 </element>
 </elements>
@@
 <via x="10.16" y="26.289" extent="1-16" drill="0.55"/>
 <wire x1="19.177" y1="54.61" x2="11.303" y2="46.736" width="0.4064" layer="1"/>
+<contactref element="B9" pad="1"/>
+<contactref element="B8" pad="1"/>
+<wire x1="13.97" y1="20.32" x2="5.08" y2="11.43" width="0.4064" layer="1"/>
+<wire x1="5.08" y1="11.43" x2="5.08" y2="7.62" width="0.4064" layer="1"/>
+<wire x1="54.61" y1="64.77" x2="60.96" y2="58.42" width="0.4064" layer="1"/>
+<wire x1="60.96" y1="58.42" x2="60.96" y2="54.61" width="0.4064" layer="1"/>
 </signal>
 <signal name="B13">
