File: HW6/ME433-EAGLE/me433-2021-1.sch (EAGLE design)
At the start: 56 parts, among them J1 B, J2 A, U2 PIC32MX170F256B

Commit message: HW10
Parts:
- added B8, B9: (no value), ME433:CONN_01
Connections:
- net B15: now also B8.1, B9.1
Changed lines of the file:
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@@
 <part name="GND21" library="ME433" deviceset="GND" device=""/>
 <part name="P+5" library="ME433" deviceset="V+" device=""/>
+<part name="B8" library="ME433" deviceset="CONN_01" device=""/>
+<part name="B9" library="ME433" deviceset="CONN_01" device=""/>
 </parts>
 <sheets>
@@
 <instance part="P+5" gate="1" x="-33.02" y="96.52" smashed="yes">
 <attribute name="VALUE" x="-30.48" y="99.06" size="1.778" layer="96" rot="R180"/>
+</instance>
+<instance part="B8" gate="G$1" x="78.74" y="48.26" smashed="yes">
+<attribute name="VALUE" x="76.2" y="43.434" size="1.778" layer="96" font="vector"/>
+<attribute name="NAME" x="73.66" y="48.768" size="1.778" layer="95" font="vector"/>
+</instance>
+<instance part="B9" gate="G$1" x="78.74" y="43.18" smashed="yes">
+<attribute name="VALUE" x="76.2" y="38.354" size="1.778" layer="96" font="vector"/>
+<attribute name="NAME" x="73.66" y="43.688" size="1.778" layer="95" font="vector"/>
 </instance>
 </instances>
@@
 <wire x1="101.6" y1="45.72" x2="91.44" y2="45.72" width="0.1524" layer="91"/>
 <label x="91.44" y="45.72" size="1.778" layer="95"/>
+<pinref part="B9" gate="G$1" pin="1"/>
+<wire x1="86.36" y1="43.18" x2="91.44" y2="43.18" width="0.1524" layer="91"/>
+<wire x1="91.44" y1="43.18" x2="91.44" y2="45.72" width="0.1524" layer="91"/>
+<pinref part="B8" gate="G$1" pin="1"/>
+<wire x1="86.36" y1="48.26" x2="91.44" y2="48.26" width="0.1524" layer="91"/>
+<wire x1="91.44" y1="48.26" x2="91.44" y2="45.72" width="0.1524" layer="91"/>
+<junction x="91.44" y="45.72"/>
 </segment>
 </net>
